File: ctrl_pcb.kicad_sch (KiCad schematic)
At the start: 28 parts, among them Q3 2N3906, Q4 2N3906, SW1 SW_D6R90, U4 TL072

Commit message: fix opampon ctrl pcb, fix accent and make slide pot slot 0.2mm wider
Parts:
- R18: value 1M -> 10k
Changed lines of the file:
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@@
     (in_bom yes) (on_board yes)
     (property "Reference" "R18" (id 0) (at 228.6 77.47 90))
-    (property "Value" "1M" (id 1) (at 228.6 80.01 90))
+    (property "Value" "10k" (id 1) (at 228.6 80.01 90))
     (property "Footprint" "ao_tht:R_Axial_DIN0207_L6.3mm_D2.5mm_P10.16mm_Horizontal" (id 2) (at 228.6 81.788 90)
       (effects (font (size 1.27 1.27)) hide)
