File: kickall.kicad_pcb (KiCad board)
At the start: 2 copper layers, 281.5 x 200 mm, 171 parts, among them J1 trig, J10 Conn_01x08_Female, J11 Conn_01x08_Male, J2 Synth_power_2x5, J3 pitch cv, J4 decay cv, J5 cv_shape, J6 accent, J7 OUT, J8 Conn_01x08_Female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

Commit message: fix opampon ctrl pcb, fix accent and make slide pot slot 0.2mm wider
Parts:
- added R79: 100k, ao_tht:R_Axial_DIN0207_L6.3mm_D2.5mm_P10.16mm_Horizontal, F.Cu at (128.0, 138.9)
- moved R77 2.03 mm to (117.9, 142.5)
- moved R76 1.78 mm to (117.9, 146.1)
- moved R61 1.52 mm to (117.9, 149.6)
- moved R64 1.27 mm to (128.0, 153.2)
- moved R75 1.27 mm to (117.9, 135.4)
- moved R72 1.02 mm to (128.0, 131.8)
- moved R62 1.02 mm to (128.0, 156.7)
- moved R67 0.76 mm to (128.0, 160.3)
- moved R73 0.76 mm to (117.9, 128.3)
- moved R70 0.51 mm to (117.9, 163.8)
Connections:
- U4 pad 5: Net-(R26-Pad1) -> GND1
- U4 pad 6: GND1 -> Net-(R26-Pad1)
Routing:
- net Net-(R75-Pad2): track 25.6 -> 31.1 mm
- net Net-(R77-Pad1): track 4.78 -> 8.76 mm
- net Net-(R74-Pad1): track 52.2 -> 55.3 mm
- net Net-(JP1-Pad1): track 28.3 -> 31.0 mm
- net Net-(R26-Pad1): track 37.1 -> 38.9 mm
- net Net-(C18-Pad2): track 69.4 -> 71.1 mm
- net Net-(J6-PadT): track 114.9 -> 116.2 mm
- net +12V: track 397.9 -> 398.9 mm
- net Net-(JP1-Pad2): track 11.4 -> 10.4 mm
- net Net-(R64-Pad2): track 4.78 -> 5.31 mm
- net Net-(J7-PadT): track 54.1 -> 53.6 mm
- net Net-(C17-Pad2): track 4.06 -> 3.56 mm
Other:
- outline, holes or cut-outs redrawn
